File: Eagle Schematic/Group12_411_REV0.sch (EAGLE design)
At the start: 13 parts, among them Q1 VN66AF

Commit message: Eagle Schematic turned In on 10/25
Parts:
- added C2, C3: (no value), resistor:C-USC0805
- added D2: ES2D, diode:ES2D
- added R3: (no value), resistor:R-US_M0805
- C1: C (none) -> 10u
- Q1: NPN (none) -> IRF530
- R1: R (none) -> 5.6k
- R2: R (none) -> 15k
Connections:
- new net N$15: OK1.A, R3.2
- new net N$17: ATMEGA328.PC2, JP1.5
- net GND: now also C2.2, C3.2
- net N$1: now also R3.1; no longer OK1.A
- net N$11: now also D2.A
- net N$3: now also C3.1, D2.C
- net VCC: now also C2.1
Other:
- note added: "FlyBack"
- note added: "This Is An Automated Plant Watering PCB"
