File: Eagle Schematic/Group12_411_REV2.sch (EAGLE design)
At the start: 23 parts, among them CN1 MiniB USB, IC1 ATMEGA32U4-AU, X1 16MHz

Commit message: For realllllzz
Parts:
- removed BOOT: EVQQ2, adaprog:EVQQ2
- removed DC1: R-78C5.0-1.0, dc-dc-converter:R-78C5.0-1.0
- removed IC1: ATMEGA32U4-AU, adaprog:ATMEGA32U4-AU
- removed ISP6: PINHD-2X3THM, adaprog:PINHD-2X3THM
- removed L: RED, adafruit:LEDCHIPLED_0805
- removed L1: 500mA, adafruit:PTCFUSE-1206
- removed PWR: GREEN, adafruit:LEDCHIPLED_0805
- removed X1: 16MHz, adaprog:XTALNX5032
- added C8: 0.1uF, adafruit:C-USC0805K
- added F1, F2: MFU0805FF00500P100, SamacSys_Parts:MFU0805FF00500P100
- added J2: 5.5x2.1mm Barrel, SparkFun-Connectors:POWER_JACKSMD
- added JP1: (no value), adafruit:PINHD-1X6-3.5MM
- added LED1, LED2: (no value), adafruit:LEDCHIP-LED0603
- added Q1: 600mA/40V, SparkFun-DiscreteSemi:TRANS_NPN-MMBT2222AL
- added R6, R7, R8: 10K, adafruit:R-US_R0805
- added S1: PTS645SM43SMTR92LFS, SamacSys_Parts:PTS645SM43SMTR92LFS
- added SV1: (no value), con-lstb:MA03-2
- added T1: 2N7002F, NXP_60_26022015:2N7002F
- added U$1: ATMEGA32U4-AU, adafruit:ATMEGA32U4-AU
- added U1: STMICROELECTRONICS_L7805ABD2T-TRSTMICROELECTRONICS_L7805ABD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, STMicroelectronics - L7805ABD2T-TR:STMICROELECTRONICS_L7805ABD2T-TRSTMICROELECTRONICS_L7805ABD2T-TR_0_0
- added X2: ABLS-16.000MHZ-B4-T, SamacSys_Parts:ABLS-16.000MHZ-B4-T
- C5: value 10uF -> 0.1uF; device adafruit:CPOL-USA/3216-18R -> adafruit:C-USC0805K
- CN1: value MiniB USB -> (none)
- R3: value 1K -> 22; R (none) -> 100
- R5: value 1K -> 22; R (none) -> 10k
Connections:
- removed net PF4: IC1.PF4(ADC4/TCK)
- removed net VBUS: CN1.VBUS, L1.1
- new net 12V: F1.2, R7.2, U1.IN
- new net N$11: Q1.C, R3.1, U$1.PD4(ICP1/ADC8)
- new net N$12: Q1.E, R5.2, U$1.PF0(ADC0)
- new net N$13: JP1.3, Q1.B
- new net N$14: JP1.2, T1.D
- new net N$15: LED2.A, R7.1
- new net N$16: F1.1, J2.PWR
- new net N$17: CN1.VBUS, F2.1
- new net N$18: R8.2, T1.G, U$1.PD5(XCK/CTS)
- new net N$19: JP1.5, U$1.PF1(ADC1)
- new net N$20: JP1.6, U$1.PD6(T1/ADC9/!OC4D)
- new net N$3: JP1.4, R3.2
- net +5V: now also F2.2, U$1.UVCC; no longer C4.1, C5.+, IC1.UVCC, IC1.VBUS, L1.2, R3.2, SJ2.2
- net GND: now also C5.2, C8.2, J2.GND, J2.GNDBREAK, LED1.C, LED2.C, R5.1, R8.1, S1.NO_1, S1.NO_2, SV1.6, T1.S, U$1.GND, U$1.GND1, U$1.GND2, U$1.GND3, U$1.UGND, U1.GND; no longer BOOT.S, BOOT.S1, C5.-, DC1.GND, IC1.GND, IC1.GND1, IC1.GND2, IC1.GND3, IC1.UGND, ISP6.6, PWR.C, R5.2
- net HWB: now also U$1.PE2(!HWB); no longer IC1.PE2(HWB)
- net MISO: now also SV1.1, U$1.PB3(PDO/MISO); no longer IC1.PB3(PDO/MISO), ISP6.1
- net MOSI: now also SV1.4, U$1.PB2(PDI/MOSI); no longer IC1.PB2(PDI/MISO), ISP6.4
- net N$1: now also SJ2.2, U$1.VBUS; no longer PWR.A, R3.1
- net N$10: now also LED1.A, R6.1; no longer L.C, R5.1
- net N$4: now also U$1.D+; no longer IC1.D+
- net N$6: now also U$1.UCAP; no longer IC1.UCAP
- net N$7: now also U$1.D-; no longer IC1.D-
- net N$8: now also U$1.XTAL1, X2.2; no longer IC1.XTAL1, X1.P$2
- net N$9: now also U$1.XTAL2, X2.1; no longer IC1.XTAL2, X1.P$1
- net PE6: now also U$1.PE6(INT.6/AIN0); no longer IC1.PE6
- net RST: now also S1.COM_1, S1.COM_2, SV1.5, U$1./RESET; no longer BOOT.P, BOOT.P1, IC1./RESET, ISP6.5
- net SCK: now also SV1.3, U$1.PB1(SCK); no longer IC1.PB1(SCK), ISP6.3
- net VCC: now also C4.1, C5.1, C8.1, JP1.1, R6.2, SV1.2, U$1.AVCC, U$1.AVCC1, U$1.VCC, U$1.VCC1, U1.OUT; no longer DC1.VOUT, IC1.AVCC, IC1.AVCC1, IC1.VCC, IC1.VCC1, ISP6.2
Other:
- note added: "Hard Ware Breakpiont"
- note added: "Power Input"
- note added: "Power LEDs"
- note added: "Reset"
- note added: "SPI Programming port"
- note removed: "http://ladyada.net/products/atmega32u4breakout/"
- moved on the sheet: C1, C2, C3, C4, C6, C7, CN1, R1, R2, R3, R4, R5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

Commit message: eagle shiz
Parts:
- renumbered U$1 to U2
Connections:
- net 12V: now also JP1.1
- net VCC: no longer JP1.1
Other:
- moved on the sheet: C2, C3, X2
