File: Eagle Schematic/Group12_411_REV3.brd (EAGLE design)
At the start: 58.4 x 45.4 mm, 32 parts, among them J2 5.5x2.1mm Barrel, Q1 600mA/40V, T1 2N7002F, U1 STMICROELECTRONICS_L7805ABD2T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, U2 ATMEGA32U4-AU, X2 ABLS-16.000MHZ-B4-T

Commit message: Cross your fingers
Parts:
- added C10: 10uF, adafruit:C0805K
- added C9: 0.1uF, adafruit:C0805K
- added R9: 100k, adafruit:R0805
- moved C6 1.27 mm to (50.8, 31.8)
Connections:
- new net N$23: C9.1, R9.1, U2.42
- new net N$25: C9.2
- net 12V: now also C10.1
- net GND: now also C10.2
- net VCC: now also R9.2
Routing:
- net N$23: track 0.00 -> 16.6 mm, vias 0 -> 2
- net VCC: track 105.3 -> 110.6 mm
- net 12V: track 81.6 -> 85.2 mm
- net N$18: track 36.3 -> 37.8 mm
- net GND: vias 15 -> 18
Other:
- board size 58.4 x 45.4 mm -> 58.4 x 45.7 mm

Commit message: Update Eagle Schematic and Board
Connect +5V on board, and add a programmable LED on pin 32 for testing
Parts:
- added LED3: (no value), adafruit:CHIP-LED0603
- added R10: 10K, adafruit:R0805
Connections:
- removed net N$25: C9.2
- new net TEST: R10.2, U2.32
- net +5V: now also SJ2.2, U2.7
- net GND: now also C9.2, LED3.C
- net N$1: now also LED3.A, R10.1; no longer SJ2.2, U2.7
Routing:
- net TEST: track 0.00 -> 34.1 mm, vias 0 -> 2
- net +5V: track 12.9 -> 39.9 mm, vias 2 -> 4
- net N$1: track 25.8 -> 3.91 mm, vias 2 -> 0
Other:
- board text added: "Automated Plant Watering System Rev. B 11/27/18"
- board text removed: "Automated Plant Watering System Rev. A 11/12/18"
Changed lines of the file:
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@@
 <text x="8.89" y="11.43" size="0.8128" layer="21" font="vector" ratio="20">Automated Plant
 Watering System
-Rev. A
-11/12/18</text>
+Rev. B
+11/27/18</text>
 <wire x1="8.89" y1="10.16" x2="7.62" y2="11.43" width="0.0254" layer="20" curve="-90"/>
 <wire x1="7.62" y1="54.61" x2="8.89" y2="55.88" width="0.0254" layer="20" curve="-90"/>
@@
 <attribute name="VALUE" x="25.67" y="47.63" size="1.016" layer="27"/>
 </element>
+<element name="R10" library="adafruit" library_urn="urn:adsk.eagle:library:420" package="R0805" package3d_urn="urn:adsk.eagle:package:6240566/1" value="10K" x="60.96" y="53.34" smashed="yes" rot="R180">
+<attribute name="NAME" x="61.722" y="52.324" size="0.8128" layer="25" rot="R180"/>
+<attribute name="R" value="1k" x="60.96" y="53.34" size="1.778" layer="27" rot="R180" display="off"/>
+<attribute name="VALUE" x="61.722" y="55.626" size="1.27" layer="27" rot="R180"/>
+</element>
+<element name="LED3" library="adafruit" library_urn="urn:adsk.eagle:library:420" package="CHIP-LED0603" package3d_urn="urn:adsk.eagle:package:6240556/1" value="" x="60.96" y="49.53" smashed="yes" rot="R90">
+<attribute name="NAME" x="61.595" y="48.895" size="0.8128" layer="25" rot="R180"/>
+<attribute name="VALUE" x="61.595" y="51.435" size="1.27" layer="27" rot="R180"/>
+</element>
 </elements>
 <signals>
@@
 <via x="40.9575" y="46.99" extent="1-16" drill="0.35"/>
 <contactref element="C10" pad="2"/>
+<contactref element="C9" pad="2"/>
+<contactref element="LED3" pad="C"/>
 </signal>
 <signal name="+5V">
@@
 <via x="26.67" y="30.48" extent="1-16" drill="0.35"/>
 <via x="31.75" y="25.4" extent="1-16" drill="0.35"/>
+<contactref element="SJ2" pad="2"/>
+<contactref element="U2" pad="7"/>
+<wire x1="19.558" y1="37.7825" x2="19.558" y2="36.068" width="0.3048" layer="1"/>
+<wire x1="19.558" y1="36.068" x2="19.05" y2="35.56" width="0.3048" layer="1"/>
+<via x="19.05" y="35.56" extent="1-16" drill="0.35"/>
+<wire x1="34.29" y1="21.59" x2="31.75" y2="24.13" width="0.3048" layer="16"/>
+<wire x1="31.75" y1="24.13" x2="20.32" y2="35.56" width="0.3048" layer="16"/>
+<wire x1="19.05" y1="35.56" x2="20.32" y2="35.56" width="0.3048" layer="16"/>
+<via x="34.29" y="21.59" extent="1-16" drill="0.35"/>
+<wire x1="34.29" y1="21.59" x2="34.29" y2="21.728628125" width="0.3048" layer="1"/>
+<wire x1="34.29" y1="21.728628125" x2="35.834465625" y2="23.27309375" width="0.3048" layer="1"/>
+<wire x1="31.75" y1="25.4" x2="31.75" y2="24.13" width="0.3048" layer="16"/>
 </signal>
 <signal name="MOSI">
@@
 <wire x1="30.48" y1="24.13" x2="32.1658875" y2="24.13" width="0.3048" layer="1"/>
 </signal>
-<signal name="N$1">
-<contactref element="SJ2" pad="2"/>
-<contactref element="U2" pad="7"/>
-<wire x1="19.558" y1="37.7825" x2="19.558" y2="36.068" width="0.3048" layer="1"/>
-<wire x1="19.558" y1="36.068" x2="19.05" y2="35.56" width="0.3048" layer="1"/>
-<via x="19.05" y="35.56" extent="1-16" drill="0.35"/>
-<wire x1="34.29" y1="21.59" x2="20.32" y2="35.56" width="0.3048" layer="16"/>
-<wire x1="19.05" y1="35.56" x2="20.32" y2="35.56" width="0.3048" layer="16"/>
-<via x="34.29" y="21.59" extent="1-16" drill="0.35"/>
-<wire x1="34.29" y1="21.59" x2="34.29" y2="21.728628125" width="0.3048" layer="1"/>
-<wire x1="34.29" y1="21.728628125" x2="35.834465625" y2="23.27309375" width="0.3048" layer="1"/>
-</signal>
 <signal name="N$2">
 <contactref element="R2" pad="1"/>
@@
 <wire x1="24.384" y1="40.624" x2="24.4" y2="40.64" width="0.3048" layer="1"/>
 </signal>
-<signal name="N$25">
-<contactref element="C9" pad="2"/>
+<signal name="TEST">
+<contactref element="U2" pad="32"/>
+<contactref element="R10" pad="2"/>
+<via x="48.26" y="35.56" extent="1-16" drill="0.35"/>
+<wire x1="41.208475" y1="34.303959375" x2="41.555240625" y2="34.303959375" width="0.3048" layer="1"/>
+<wire x1="41.555240625" y1="34.303959375" x2="42.0014625" y2="34.75018125" width="0.3048" layer="1"/>
+<wire x1="47.45018125" y1="34.75018125" x2="48.26" y2="35.56" width="0.3048" layer="1"/>
+<wire x1="42.0014625" y1="34.75018125" x2="47.45018125" y2="34.75018125" width="0.3048" layer="1"/>
+<wire x1="48.26" y1="35.56" x2="48.26" y2="38.1" width="0.3048" layer="16"/>
+<wire x1="48.26" y1="38.1" x2="50.8" y2="40.64" width="0.3048" layer="16"/>
+<via x="50.8" y="40.64" extent="1-16" drill="0.35"/>
+<wire x1="50.8" y1="40.64" x2="50.8" y2="50.8" width="0.3048" layer="1"/>
+<wire x1="50.8" y1="50.8" x2="53.34" y2="53.34" width="0.3048" layer="1"/>
+<wire x1="53.34" y1="53.34" x2="59.96" y2="53.34" width="0.3048" layer="1"/>
+</signal>
+<signal name="N$1">
+<contactref element="R10" pad="1"/>
+<contactref element="LED3" pad="A"/>
+<wire x1="61.96" y1="53.34" x2="61.96" y2="49.78" width="0.3048" layer="1"/>
+<wire x1="61.96" y1="49.78" x2="61.71" y2="49.53" width="0.3048" layer="1"/>
 </signal>
 </signals>
